Commit message: Add velocity controllers

File: kortex_description/arms/gen3/7dof/urdf/gen3_transmission_macro.xacro (robot description, xacro)
@@ -2,5 +2,5 @@
 <robot xmlns:xacro="http://ros.org/wiki/xacro">
     <xacro:macro name="load_gazebo_arm_transmissions" params="prefix">
-        <transmission name="${prefix}joint_1_transmission">
+        <!--transmission name="${prefix}joint_1_transmission">
         <type>transmission_interface/SimpleTransmission</type>
         <joint name="${prefix}joint_1">
@@ -64,4 +64,67 @@
             <mechanicalReduction>1</mechanicalReduction>
         </actuator>
+        </transmission-->
+        <transmission name="${prefix}joint_1_transmission">
+        <type>transmission_interface/SimpleTransmission</type>
+        <joint name="${prefix}joint_1">
+            <hardwareInterface>hardware_interface/VelocityJointInterface</hardwareInterface>
+        </joint>
+        <actuator name="${prefix}joint_1_motor">
+            <mechanicalReduction>1</mechanicalReduction>
+        </actuator>
+        </transmission>
+        <transmission name="${prefix}joint_2_transmission">
+        <type>transmission_interface/SimpleTransmission</type>
+        <joint name="${prefix}joint_2">
+            <hardwareInterface>hardware_interface/VelocityJointInterface</hardwareInterface>
+        </joint>
+        <actuator name="${prefix}joint_2_motor">
+            <mechanicalReduction>1</mechanicalReduction>
+        </actuator>
+        </transmission>
+        <transmission name="${prefix}joint_3_transmission">
+        <type>transmission_interface/SimpleTransmission</type>
+        <joint name="${prefix}joint_3">
+            <hardwareInterface>hardware_interface/VelocityJointInterface</hardwareInterface>
+        </joint>
+        <actuator name="${prefix}joint_3_motor">
+            <mechanicalReduction>1</mechanicalReduction>
+        </actuator>
+        </transmission>
+        <transmission name="${prefix}joint_4_transmission">
+        <type>transmission_interface/SimpleTransmission</type>
+        <joint name="${prefix}joint_4">
+            <hardwareInterface>hardware_interface/VelocityJointInterface</hardwareInterface>
+        </joint>
+        <actuator name="${prefix}joint_4_motor">
+            <mechanicalReduction>1</mechanicalReduction>
+        </actuator>
+        </transmission>
+        <transmission name="${prefix}joint_5_transmission">
+        <type>transmission_interface/SimpleTransmission</type>
+        <joint name="${prefix}joint_5">
+            <hardwareInterface>hardware_interface/VelocityJointInterface</hardwareInterface>
+        </joint>
+        <actuator name="${prefix}joint_5_motor">
+            <mechanicalReduction>1</mechanicalReduction>
+        </actuator>
+        </transmission>
+        <transmission name="${prefix}joint_6_transmission">
+        <type>transmission_interface/SimpleTransmission</type>
+        <joint name="${prefix}joint_6">
+            <hardwareInterface>hardware_interface/VelocityJointInterface</hardwareInterface>
+        </joint>
+        <actuator name="${prefix}joint_6_motor">
+            <mechanicalReduction>1</mechanicalReduction>
+        </actuator>
+        </transmission>
+        <transmission name="${prefix}joint_7_transmission">
+        <type>transmission_interface/SimpleTransmission</type>
+        <joint name="${prefix}joint_7">
+            <hardwareInterface>hardware_interface/VelocityJointInterface</hardwareInterface>
+        </joint>
+        <actuator name="${prefix}joint_7_motor">
+            <mechanicalReduction>1</mechanicalReduction>
+        </actuator>
         </transmission>
     </xacro:macro>
